File: KiCAD/TeensyVariety/TeensyVariety.kicad_sch (KiCad schematic)
At the start: 36 parts, among them J1 CH1, J2 TRIG INP, J3 LASER, J4 CH2, J5 CH3, J6 CH4 / Decimated Trig, J7 DEBUG, J8 PHOTOTRANSISTOR, Q2 Q_NPN_BCE, U1 Teensy4.0

Commit message: Updated UI and also minor edits to unfinished PCB
Parts:
- added R13: 10R, Resistor_SMD:R_0805_2012Metric, symbol Device:R
- R2: value 1K -> 6.7K
Connections:
- net Laser -: now also R13.1; no longer Q2.2 (C)
- new net: Q2.2 (C), R13.2
Changed lines of the file:
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@@
-	(wire
-		(pts
-			(xy 143.51 119.38) (xy 158.75 119.38)
-		)
-		(stroke
-			(width 0)
-			(type default)
-		)
-	)
 	(wire
 		(pts
@@
 	(wire
 		(pts
+			(xy 143.51 119.38) (xy 143.51 121.92)
+		)
+		(stroke
+			(width 0)
+			(type default)
+		)
+	)
+	(wire
+		(pts
 			(xy 116.84 154.94) (xy 120.65 154.94)
 		)
@@
 	(wire
 		(pts
-			(xy 143.51 121.92) (xy 143.51 119.38)
+			(xy 158.75 119.38) (xy 151.13 119.38)
 		)
 		(stroke
@@
 			)
 		)
-		(property "Value" "1K"
+		(property "Value" "6.7K"
 			(at 132.08 123.19 90)
 			(effects
@@
 					(unit 1)
 				)
+			)
+		)
+	)
+	(symbol
+		(lib_id "Device:R")
+		(at 147.32 119.38 270)
+		(unit 1)
+		(exclude_from_sim no)
+		(in_bom yes)
+		(on_board yes)
+		(dnp no)
+		(fields_autoplaced yes)
+		(property "Reference" "R13"
+			(at 147.32 113.03 90)
+			(effects
+				(font
+					(size 1.27 1.27)
+				)
+			)
+		)
+		(property "Value" "10R"
+			(at 147.32 115.57 90)
+			(effects
+				(font
+					(size 1.27 1.27)
+				)
+			)
+		)
+		(property "Footprint" "Resistor_SMD:R_0805_2012Metric"
+			(at 147.32 117.602 90)
+			(effects
+				(font
+					(size 1.27 1.27)
+				)
+				(hide yes)
+			)
+		)
+		(property "Datasheet" "~"
+			(at 147.32 119.38 0)
+			(effects
+				(font
+					(size 1.27 1.27)
+				)
+				(hide yes)
+			)
+		)
+		(property "Description" "Resistor"
+			(at 147.32 119.38 0)
+			(effects
+				(font
+					(size 1.27 1.27)
+				)
+				(hide yes)
+			)
+		)
+		(pin "1"
+		)
+		(pin "2"
+		)
+		(instances
+			(project "TeensyVariety"
+				(path "/2fb4ce1b-d967-452b-a6a8-6c10cc605e92"
+					(reference "R13")
+					(unit 1)
+				)
